File: hardware/Kompic_Mk1/Kompic_Mk1.kicad_sch (KiCad schematic)
At the start: 0 parts

Commit message: Added Circuit page! Minor touchups to schematic + Schematic PDF.
Other:
- company: Ivan Porupski May2026(c) -> Ivan Porupski June2026(c)
Changed lines of the file:
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@@
 	(title_block
 		(title "Kompić Mk1")
-		(date "2026-05-30")
-		(rev "iv7.0")
-		(company "Ivan Porupski May2026(c)")
+		(date "2026-06-02")
+		(rev "iv7.1")
+		(company "Ivan Porupski June2026(c)")
 	)
 	(sheet
