File: hardware/Kompic_Mk1/1_ESP32-S3_Wroom.kicad_sch (KiCad schematic)
At the start: 39 parts, among them J1 Conn_02x12_Top_Bottom, J2 MB Interface, SW2 EC05E1220401, U1 ESP32-S3-WROOM-1U-N16R8

Commit message: BIG CHANGE: Had bad wiring for the AMOLED, had to redo the schematic and complete routing of PCB (iv7.1). Added Arduino sketch for verifying AMOLED. Added newly redone pinout for both ESP32-S3 and the AMOLED.
Parts:
- removed J1: Conn_02x12_Top_Bottom, New_Library:Connector_b2b_OK-F024-04_v1, symbol Connector_Generic:Conn_02x12_Top_Bottom
- removed TP22: QSPI_TE, TestPoint:TestPoint_Pad_D1.0mm, symbol Connector:TestPoint
- added J1: Conn_02x12_OK-14F024-04_v1, New_Library:Connector_b2b_OK-F024-04_v1, symbol New_Library:Conn_02x12_OK-14F024-04_v1
Connections:
- net OLED_EN is gone; now on net QSPI_TE: U1.26 (IO45)
- net +3V3: now also J1.12 (Pin_12), J1.14 (Pin_14), J1.3 (Pin_3), J1.5 (Pin_5), J1.6 (Pin_6)
- net GND: now also J1.2 (Pin_2), J1.20 (Pin_20), J1.22 (Pin_22), J1.24 (Pin_24), J1.27 (Pin_27), J1.28 (Pin_28), J1.29 (Pin_29), J1.30 (Pin_30), J1.7 (Pin_7)
- net MAX_INT: now also U1.7 (IO7); no longer U1.18 (IO10)
- net QSPI-CLK: now also J1.21 (Pin_21)
- net QSPI-I1: now also J1.15 (Pin_15)
- net QSPI-I2: now also J1.17 (Pin_17)
- net QSPI-I3: now also J1.19 (Pin_19)
- net QSPI-IO: now also J1.23 (Pin_23)
- net QSPI-RESET: now also J1.1 (Pin_1)
- net QSPI_CS: now also U1.18 (IO10), J1.16 (Pin_16); no longer U1.16 (IO46)
- net QSPI_TE: now also J1.13 (Pin_13)
- net SCL: now also J1.11 (Pin_11)
- net SDA: now also J1.10 (Pin_10)
- net TP-INT_3V3: now also J1.9 (Pin_9)
- net TP-RST_3V3: now also J1.8 (Pin_8)
- net TimePulse: now also U1.16 (IO46); no longer U1.7 (IO7)
- no-connect marks 0 -> 2
Other:
- note removed: "VBAT expects min 3.5V"
- moved on the sheet: TP15, TP23

Commit message: Added Circuit page! Minor touchups to schematic + Schematic PDF.
Other:
- company: Ivan Porupski May2026(c) -> Ivan Porupski June2026(c)
Changed lines of the file:
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@@
 	(paper "A4")
 	(title_block
-		(date "2026-05-30")
+		(date "2026-06-02")
 		(rev "iv7.1")
-		(company "Ivan Porupski May2026(c)")
+		(company "Ivan Porupski June2026(c)")
 	)
 	(text "2.06-inch AMOLED\n(CO5300AF-51+CST9217)\nOK-14F024-04 connector"

Commit message: MASSIVE UPDATE: Built a working prototype with most systems go! iv7.1 requires about half a dozen surgical hacks on the PCB itself - it is suggested you wait for iv7.2+ - but otherwise, a massive success!
Stage 1-3 documents how the parts were added, in what fashion and then tested both electrically and with the scripts in test/ for each stage. SD Card may be unfixable in iv7.1.

Added notes where the bugs are in the schematic, but haven't updated it.
Other:
- note added: "BUG: CLK MISSING 10k PULLUP"
- note added: "BUG: CMD and DAT to 5k1 (4k7)"
Changed lines of the file:
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@@
+		)
+	)
+	(text "BUG: CLK MISSING 10k PULLUP"
+		(exclude_from_sim no)
+		(at 236.728 112.014 0)
+		(effects
+			(font
+				(size 2.54 2.54)
+				(thickness 0.508)
+				(bold yes)
+				(color 255 38 26 1)
+			)
+		)
+	)
+	(text "BUG: CMD and DAT to 5k1 (4k7)"
+		(exclude_from_sim no)
+		(at 230.886 119.888 0)
+		(effects
+			(font
+				(size 2.54 2.54)
+				(thickness 0.508)
+				(bold yes)
+				(color 255 38 26 1)
+			)
 		)
 	)
