File: hardware/Kompic_Mk1/1_ESP32-S3_Wroom.kicad_sch (KiCad schematic)
At the start: 38 parts, among them J1 Conn_02x12_OK-14F024-04_v1, J2 MB Interface, SW2 EC05E1220401, U1 ESP32-S3-WROOM-1U-N16R8

Commit message: hardware: Kompic Mk1 schematic edits + TDFN-8 footprint; Mk1b PCB start
Mk1: LCSC parts refresh, ESP32-S3 sheet edits, project file bump,
symbol library tweak, new TDFN-8 (2.0x2.0 P0.50 EP1.2) footprint +
STEP + WRL for the sensor package used on Mk1b.

Mk1b: fresh PCB project seeded from Mk1 with the AMOLED receptacle
footprint mirror fix from Stage 16.
Other:
- note added: "CRITICAL BUG: Connector wired in mirror!!!"
Changed lines of the file:
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@@
+		)
+	)
+	(text "CRITICAL BUG: Connector wired in mirror!!!"
+		(exclude_from_sim no)
+		(at 55.626 156.972 0)
+		(effects
+			(font
+				(size 2.54 2.54)
+				(thickness 0.508)
+				(bold yes)
+				(color 255 38 26 1)
+			)
 		)
 	)
