File: hardware/Kompic_Mk1/4_Air_Sensors.kicad_sch (KiCad schematic)
At the start: 5 parts, among them U10 MSM261DGT003, U9 BME688_C3664478

Commit message: Added Circuit page! Minor touchups to schematic + Schematic PDF.
Other:
- company: Ivan Porupski May2026(c) -> Ivan Porupski June2026(c)
Changed lines of the file:
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@@
 	(paper "A4")
 	(title_block
-		(date "2026-05-30")
-		(rev "iv7.0")
-		(company "Ivan Porupski May2026(c)")
+		(date "2026-06-02")
+		(rev "iv7.1")
+		(company "Ivan Porupski June2026(c)")
 	)
 	(text "Air Quality (BME688)"

Commit message: MASSIVE UPDATE: Built a working prototype with most systems go! iv7.1 requires about half a dozen surgical hacks on the PCB itself - it is suggested you wait for iv7.2+ - but otherwise, a massive success!
Stage 1-3 documents how the parts were added, in what fashion and then tested both electrically and with the scripts in test/ for each stage. SD Card may be unfixable in iv7.1.

Added notes where the bugs are in the schematic, but haven't updated it.
Other:
- note added: "BUG: VDD SHOULD BE 3V3; 1V8 LEAKBACK"
Changed lines of the file:
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@@
+		)
+	)
+	(text "BUG: VDD SHOULD BE 3V3; 1V8 LEAKBACK"
+		(exclude_from_sim no)
+		(at 235.204 99.568 0)
+		(effects
+			(font
+				(size 2.54 2.54)
+				(thickness 0.508)
+				(bold yes)
+				(color 255 38 26 1)
+			)
 		)
 	)
