File: hardware/Kompic_Mk1/Kompic_Mk1.kicad_pcb (KiCad board)
At the start: 4 copper layers, 44.5 x 50.6 mm, 144 parts, among them CN1 Qvar_Electrode_2, CN2 Qvar_Electrode_1, J1 Conn_02x12_OK-14F024-04_v1, J2 MB Interface, J3 DB-Interface, M1 ELV1411A, SW1 SKSCLBE010, SW2 EC05E1220401, U1 ESP32-S3-WROOM-1U-N16R8, U10 MSM261DGT003, U11 VEML6030, U12 BSS138W_C890266, U13 MAX30101EFD+T, U14 DRV2605LDGSR, U15 TMP117AIDRVR, U16 TPS62840DLCR, U2 XC6206P182MR, U4 BQ25619RTWR, U5 LSM6DSV16XTR, U6 MAX-M10S-00B, U7 LIS3MDLTR, U8 PCF85063ATL/1,118, U9 BME688_C3664478, X1 FC31M2-32.768-NTLLLDT

Commit message: Massive progress: Folder restructuring of firmware/ to harbor arduino sketches and the esp-idf main project. Working demos. Building notes in the 5-6 Stage reports.
Other:
- board text added: "2x FLASHLIGHT CUTS"
- board text added: "CUT 1v8 BRANCH"
Changed lines of the file:
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@@
+	)
+	(gr_line
+		(start 172.1 103.8)
+		(end 172.1 105.7)
+		(stroke
+			(width 0.3)
+			(type solid)
+		)
+		(layer "Eco2.User")
+	)
+	(gr_line
+		(start 174.2 116.05)
+		(end 176 116.8)
+		(stroke
+			(width 0.3)
+			(type solid)
+		)
+		(layer "Eco2.User")
+	)
+	(gr_line
+		(start 174.8 110.85)
+		(end 174.8 112.75)
+		(stroke
+			(width 0.3)
+			(type solid)
+		)
+		(layer "Eco2.User")
 	)
 	(gr_line
@@
 			)
 			(justify left bottom)
+		)
+	)
+	(gr_text "CUT 1v8 BRANCH"
+		(at 166.8 102.9 0)
+		(layer "Eco2.User")
+		(effects
+			(font
+				(size 1 1)
+				(thickness 0.15)
+			)
+			(justify left bottom)
+		)
+	)
+	(gr_text "2x FLASHLIGHT\nCUTS"
+		(at 177.5 116.4 0)
+		(layer "Eco2.User")
+		(effects
+			(font
+				(size 1 1)
+				(thickness 0.15)
+			)
+			(justify left bottom)
