File: hardware/Kompic_Mk1b/3_Space_Time_Sensors.kicad_sch (KiCad schematic)
At the start: 37 parts, among them CN1 Qvar_Electrode_2, U5 LSM6DSV16XTR, U6 MAX-M10S-00B, U7 LIS3MDLTR, U8 PCF85063ATL/1,118, X1 FC31M2-32.768-NTLLLDT

Commit message: firmware: Stage 30 close + Stage 31 plan checkpoint (fw 0.4.75)
Stage 30 shipped: esp_lvgl_port + PARTIAL refresh restored, sleep-race
mutex, AUTOSHDN CLI+NVS, NVS dump verb, FLASH bypass verb, landscape
+ Mode HUD deferred to Stage 31 per foundations-rebuild plan.

Stage docs 24-30 landed (Mk1b bring-up through display port migration),
Stage 31 (LVGL foundations rebuild plan) and Stage 34 (naming + CLI
restructure) opened. LOG.md + LOG_TAGS.md loose-ends surfaces added.

Component surgery in this checkpoint:
  - co5300 split: co5300.c -> co5300_panel.{c,h} + co5300_panel_io.{c,h}
  - qvar_ecg deleted (NO ECG on Kompic)
  - max17048 new component (fuel gauge on Mk1b)
  - *_cmd.c extracts landed for bq25619/drv2605/encoder/pcf85063/
    veml6030/ws2812 per Module_Blueprint two-outlet pattern
  - Encoder-dead stopgap: field_capture boots to FCM_FLASHLIGHT
    (does not persist; revert once encoder fix lands)

Hardware: Mk1b sch/pcb touch-ups (3_Space_Time_Sensors).

Arduino field-demo sketches 16/17/18 (amoled+touch / max17048 / GPS)
landed as freeze-and-forget references per arduino-sketch-pattern.

Mk2_intel folder seeded (Mk1+Mk1b field learnings for Mk2 fab wait).

Bare-working checkpoint before Stage 31.1 (shared pane style) starts.

Co-Authored-By: Claude Opus 4.7 <noreply@anthropic.com>
Other:
- note added: "BUG: pin 15 V_SET should be FLOATING"
- note added: "BUG: pin 7 V_io should be FLOATING"
- note added: "BUG: pins 17 SCL and 16 SDA SHOULD BE FLOATING"
Changed lines of the file:
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@@
+		)
+	)
+	(text "BUG:  pin 7 V_io should be FLOATING"
+		(exclude_from_sim no)
+		(at 62.23 185.928 0)
+		(effects
+			(font
+				(size 2.032 2.032)
+				(thickness 0.4064)
+				(bold yes)
+				(color 255 31 41 1)
+			)
 		)
 	)
@@
 				(thickness 0.762)
 				(bold yes)
+			)
+		)
+	)
+	(text "BUG:  pin 15 V_SET should be FLOATING"
+		(exclude_from_sim no)
+		(at 167.386 148.59 0)
+		(effects
+			(font
+				(size 2.032 2.032)
+				(thickness 0.4064)
+				(bold yes)
+				(color 255 31 41 1)
 			)
 		)
@@
 			)
 		)
+	)
+	(text "BUG: pins 17 SCL and 16 SDA SHOULD BE FLOATING"
+		(exclude_from_sim no)
+		(at 140.716 134.366 0)
+		(effects
+			(font
+				(size 2.032 2.032)
+				(thickness 0.4064)
+				(bold yes)
+				(color 255 31 41 1)
+			)
+		)
