File: hardware/Kompic_Mk1b/Kompic_Mk1b.kicad_pcb (KiCad board)
At the start: 4 copper layers, 44.5 x 50.6 mm, 149 parts, among them CN1 Qvar_Electrode_2, CN2 Qvar_Electrode_1, J1 Conn_02x12_OK-14F024-04_v1, J2 MB Interface, J3 DB-Interface, M1 ELV1411A, SW1 SKSCLBE010, SW2 EC05E1220401, U1 ESP32-S3-WROOM-1U-N16R8, U10 MSM261DGT003, U11 VEML6030, U12 BSS138W_C890266, U13 MAX30101EFD+T, U14 DRV2605LDGSR, U15 TMP117AIDRVR, U16 TPS62840DLCR, U2 XC6206P182MR, U3 MAX17048G+T10, U4 BQ25619RTWR, U5 LSM6DSV16XTR, U6 MAX-M10S-00B, U7 LIS3MDLTR, U8 PCF85063ATL/1,118, U9 BME688_C3664478, X1 FC31M2-32.768-NTLLLDT

Commit message: firmware: Stage 30 close + Stage 31 plan checkpoint (fw 0.4.75)
Stage 30 shipped: esp_lvgl_port + PARTIAL refresh restored, sleep-race
mutex, AUTOSHDN CLI+NVS, NVS dump verb, FLASH bypass verb, landscape
+ Mode HUD deferred to Stage 31 per foundations-rebuild plan.

Stage docs 24-30 landed (Mk1b bring-up through display port migration),
Stage 31 (LVGL foundations rebuild plan) and Stage 34 (naming + CLI
restructure) opened. LOG.md + LOG_TAGS.md loose-ends surfaces added.

Component surgery in this checkpoint:
  - co5300 split: co5300.c -> co5300_panel.{c,h} + co5300_panel_io.{c,h}
  - qvar_ecg deleted (NO ECG on Kompic)
  - max17048 new component (fuel gauge on Mk1b)
  - *_cmd.c extracts landed for bq25619/drv2605/encoder/pcf85063/
    veml6030/ws2812 per Module_Blueprint two-outlet pattern
  - Encoder-dead stopgap: field_capture boots to FCM_FLASHLIGHT
    (does not persist; revert once encoder fix lands)

Hardware: Mk1b sch/pcb touch-ups (3_Space_Time_Sensors).

Arduino field-demo sketches 16/17/18 (amoled+touch / max17048 / GPS)
landed as freeze-and-forget references per arduino-sketch-pattern.

Mk2_intel folder seeded (Mk1+Mk1b field learnings for Mk2 fab wait).

Bare-working checkpoint before Stage 31.1 (shared pane style) starts.

Co-Authored-By: Claude Opus 4.7 <noreply@anthropic.com>
Other:
- board text added: "Should be floating for 3v2, or gnd for 1v8"
- board text added: "needs jumper 1v8 to daughter board"
Changed lines of the file:
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@@
+	)
+	(gr_line
+		(start 159.395 94.86)
+		(end 166.5 94.8)
+		(stroke
+			(width 0.5)
+			(type solid)
+		)
+		(layer "Eco2.User")
+	)
+	(gr_line
+		(start 159.75 90.3)
+		(end 161.25 90.3)
+		(stroke
+			(width 0.5)
+			(type solid)
+		)
+		(layer "Eco2.User")
+	)
+	(gr_line
+		(start 159.95 92.8)
+		(end 161.45 92.8)
+		(stroke
+			(width 0.5)
+			(type solid)
+		)
+		(layer "Eco2.User")
+	)
+	(gr_line
+		(start 163.1 99.9)
+		(end 164.6 99.9)
+		(stroke
+			(width 0.5)
+			(type solid)
+		)
+		(layer "Eco2.User")
+	)
+	(gr_line
+		(start 163.1 102.2)
+		(end 164.6 102.2)
+		(stroke
+			(width 0.5)
+			(type solid)
+		)
+		(layer "Eco2.User")
 	)
 	(gr_line
@@
 		)
 	)
+	(gr_text "needs jumper 1v8 to daughter board"
+		(at 165.1 98.4 0)
+		(layer "Eco2.User")
+		(effects
+			(font
+				(size 1 1)
+				(thickness 0.15)
+			)
+			(justify left bottom)
+		)
+	)
+	(gr_text "Should be floating for 3v2, or gnd for 1v8"
+		(at 160.65 92.7 45)
+		(layer "Eco2.User")
+		(effects
+			(font
+				(size 1 1)
+				(thickness 0.15)
+			)
+			(justify left bottom)
+		)
+	)
