File: hardware/Kompic_Mk1b/Kompic_Mk1b.kicad_pcb (KiCad board)
At the start: 4 copper layers, 44.5 x 50.6 mm, 149 parts, among them CN1 Qvar_Electrode_2, CN2 Qvar_Electrode_1, J1 Conn_02x12_OK-14F024-04_v1, J2 MB Interface, J3 DB-Interface, M1 ELV1411A, SW1 SKSCLBE010, SW2 EC05E1220401, U1 ESP32-S3-WROOM-1U-N16R8, U10 MSM261DGT003, U11 VEML6030, U12 BSS138W_C890266, U13 MAX30101EFD+T, U14 DRV2605LDGSR, U15 TMP117AIDRVR, U16 TPS62840DLCR, U2 XC6206P182MR, U3 MAX17048G+T10, U4 BQ25619RTWR, U5 LSM6DSV16XTR, U6 MAX-M10S-00B, U7 LIS3MDLTR, U8 PCF85063ATL/1,118, U9 BME688_C3664478, X1 FC31M2-32.768-NTLLLDT

Commit message: Final firmware changes; GPS hardware fixing and arduino sketches (18, 19); Started progress on migrating to LVGL 9 optimized architecture.
Other:
- board text added: "SAFEBOOT -> FLOAT SDA/SCL not in use -> FLOAT"
Changed lines of the file:
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@@
+	)
+	(gr_line
+		(start 156.2 94.6)
+		(end 158.5 94.6)
+		(stroke
+			(width 0.5)
+			(type solid)
+		)
+		(layer "Eco1.User")
+	)
+	(gr_line
+		(start 160 94.6)
+		(end 162.3 94.6)
+		(stroke
+			(width 0.5)
+			(type solid)
+		)
+		(layer "Eco1.User")
+	)
+	(gr_line
+		(start 163.8 94.6)
+		(end 166.1 94.6)
+		(stroke
+			(width 0.5)
+			(type solid)
+		)
+		(layer "Eco1.User")
 	)
 	(gr_line
@@
 		)
 	)
+	(gr_text "SAFEBOOT -> FLOAT\nSDA/SCL not in use -> FLOAT"
+		(at 140.8 96 0)
+		(layer "Eco1.User")
+		(effects
+			(font
+				(size 1 1)
+				(thickness 0.15)
+			)
+			(justify left bottom)
+		)
+	)
